File: eagle/avr.brd (EAGLE design)
At the start: 74.6 x 48.2 mm, 22 parts, among them IC1 MEGA8-P, IC2 7805TV, Q1 16MHz

Commit message: Updated pinouts
Parts:
- removed C6: 0.1uF, resistor:C050-025X075
- removed C7: (no value), resistor:C050-025X075
- added 3.3V: LD115A-3.3v, linear:TO220V
- added C8: 0.1uF, resistor:C050-025X075
- added C9: 10uF, resistor:C050-025X075
- ETHER: device pinhead:1X10 -> pinhead:2X05
Connections:
- net N$1 renamed +12V
- removed net CLKOUT: ETHER.10
- new net +3V3: 3.3V.3, C9.1, RFID.8
- new net CLK_OUT: ETHER.1
- net +5V: now also 3.3V.1, C8.1, ETHER.9; no longer C6.1, C7.1, ETHER.5, RFID.6
- net ETHER_INT: now also ETHER.2; no longer ETHER.1
- net GND: now also 3.3V.2, C8.2, C9.2, ETHER.10, RFID.6; no longer C6.2, C7.2, ETHER.6, RFID.8
- net MISO: now also ETHER.4, RFID.3; no longer ETHER.2, RFID.4
- net MOSI: now also ETHER.5, RFID.4; no longer ETHER.8, RFID.3
- net RESET: now also ETHER.8; no longer ETHER.4
- net SCK: now also ETHER.6; no longer ETHER.3
- net WOL: now also ETHER.3; no longer ETHER.9
Routing:
- net MISO: track 85.6 -> 58.1 mm
- net +5V: track 109.1 -> 88.5 mm
- net MOSI: track 67.9 -> 54.1 mm
- net RESET: track 115.2 -> 106.3 mm
- net ETHER_INT: track 32.9 -> 26.5 mm
- net CS_ETHER: track 37.7 -> 31.3 mm
- net SCK: track 70.6 -> 69.3 mm
